File: Control.sch (KiCad schematic (older format))
At the start: 27 parts, among them IC1 ATMEGA16A-P, P6 Switch, P7 CONN_01X06, X1 12Mhz

Commit message: Changes to be committed: 	new file:   78LXXSOT89.pdf 	modified:   Control.sch 	modified:   Debugger.sch 	modified:   MotorDriver.sch 	modified:   PS.sch 	modified:   Sensor.sch 	new file:   XL6009-Schematic-Diagram.pdf 	modified:   main-cache.lib 	new file:   main.cmp 	new file:   main.kicad_pcb 	new file:   main.net 	modified:   main.pro 	modified:   main.sch
Parts:
- removed D1: RGB, symbol LED_RGB
- removed S1, S2, S3: SW, symbol SW_TACT
- added D1: RED, LEDs:LED-3MM, symbol LED
- added D2: BLUE, LEDs:LED-3MM, symbol LED
- added D3: GREEN, LEDs:LED-3MM, symbol LED
- added SW1, SW2, SW3, SW4, SW5: SW_PUSH, Pin_Headers:Pin_Header_Straight_1x02, symbol SW_PUSH
- C1, C2, C3, C5: footprint (none) -> Capacitors_SMD:C_0805_HandSoldering
- C4, L1: footprint (none) -> Capacitors_ThroughHole:Capacitor5x6RM2.5
- DS1: footprint WC1602A -> Socket_Strips:Socket_Strip_Straight_1x16
- IC1: footprint DIL40 -> Sockets_DIP:DIP-40__600_ELL
- P4: renamed from P6; footprint (none) -> Pin_Headers:Pin_Header_Straight_2x02
- P5: renamed from P7; value CONN_01X06 -> ISP; footprint (none) -> Pin_Headers:Pin_Header_Straight_1x06
- R1, R10, R11, R2, R3, R4, R5, R7, R8, R9: footprint (none) -> Resistors_SMD:R_0805_HandSoldering
- R6: value R -> 1K; footprint (none) -> Resistors_SMD:R_0805_HandSoldering
- RV1: footprint (none) -> Potentiometers:Potentiometer_Trimmer-Suntan-TSR-3386P
- X1: footprint (none) -> Crystals:Crystal_HC49-U_Vertical
Connections:
- net labels added: ADC[0..4]
- net labels removed: ADC
- wire segments 128 -> 129
Other:
- moved on the sheet: C1, C2, C3, C4, C5, DS1, IC1, L1, P4, P5, R1, R10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

Commit message: update
Parts:
- DS1: footprint Socket_Strips:Socket_Strip_Straight_1x16 -> display-lcd:TUXGR_16X2_R2
- R6: footprint Resistors_SMD:R_0805_HandSoldering -> Resistors_ThroughHole:Resistor_Horizontal_RM15mm
- RV1: footprint Potentiometers:Potentiometer_Trimmer-Suntan-TSR-3386P -> Potentiometers:Potentiometer_Triwood_RM-065
Connections:
- net GND: now also RV1.1; no longer RV1.3
- net VCC: now also RV1.3; no longer RV1.1
Changed lines of the file:
@@
 LIBS:memory
 LIBS:xilinx
-LIBS:special
 LIBS:microcontrollers
 LIBS:dsp
@@
 encoding utf-8
 Sheet 3 6
-Title ""
-Date ""
-Rev ""
+Title "KENZANIN LINEFOLLOWER"
+Date "2015-06-28"
+Rev "1.0"
 Comp ""
 Comment1 ""
@@
 F 0 "DS1" H 5600 2550 40  0000 C CNN
 F 1 "LCD16X2" H 7100 2550 40  0000 C CNN
-F 2 "Socket_Strips:Socket_Strip_Straight_1x16" H 6400 2100 35  0001 C CIN
+F 2 "display-lcd:TUXGR_16X2_R2" H 6400 2100 35  0001 C CIN
 F 3 "" H 6400 2150 60  0000 C CNN
 	1    6400 2150
@@
 F 0 "RV1" H 6950 3950 50  0000 C CNN
 F 1 "POT" H 6950 4050 50  0000 C CNN
-F 2 "Potentiometers:Potentiometer_Trimmer-Suntan-TSR-3386P" H 6950 4050 60  0001 C CNN
+F 2 "Potentiometers:Potentiometer_Triwood_RM-065" H 6950 4050 60  0001 C CNN
 F 3 "" H 6950 4050 60  0000 C CNN
 	1    6950 4050
@@
 L GND #PWR06
 U 1 1 558C556D
-P 6650 4050
-F 0 "#PWR06" H 6650 4050 30  0001 C CNN
-F 1 "GND" H 6650 3980 30  0001 C CNN
-F 2 "" H 6650 4050 60  0000 C CNN
-F 3 "" H 6650 4050 60  0000 C CNN
-	1    6650 4050
-	0    1    -1   0
-$EndComp
-Text HLabel 7250 4050 2    60   UnSpc ~ 0
+P 7250 4050
+F 0 "#PWR06" H 7250 4050 30  0001 C CNN
+F 1 "GND" H 7250 3980 30  0001 C CNN
+F 2 "" H 7250 4050 60  0000 C CNN
+F 3 "" H 7250 4050 60  0000 C CNN
+	1    7250 4050
+	0    -1   1    0
+$EndComp
+Text HLabel 6650 4050 0    60   UnSpc ~ 0
 VCC
 Wire Wire Line
@@
 F 0 "R6" V 5730 3000 40  0000 C CNN
 F 1 "1K" V 5657 3001 40  0000 C CNN
-F 2 "Resistors_SMD:R_0805_HandSoldering" V 5580 3000 30  0001 C CNN
+F 2 "Resistors_ThroughHole:Resistor_Horizontal_RM15mm" V 5580 3000 30  0001 C CNN
 F 3 "" H 5650 3000 30  0000 C CNN
 	1    5650 3000
