File: main.kicad_pcb (KiCad board)
At the start: 2 copper layers, 51 parts, among them IC1 ATMEGA16A-P, P1 MA, P2 MA, P3 MB, P4 Switch, P5 ISP, P6 5V, P7 12V, P8 SERIAL, P9 POWER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

Commit message: update
Parts:
- removed Q1: 2N2222, Discret:TO92PN
- removed R12: 8K3, Resistors_SMD:R_0805_HandSoldering
- removed R13: 33K, Resistors_SMD:R_0805_HandSoldering
- removed R14: 220R, Resistors_SMD:R_0805_HandSoldering
- removed RP1: 4K7, Pin_Arrays:pin_array_1x06
- removed U3, U4, U5: TCRT5000, TCRT5000:TCRT5000
- removed U6: 78L33, Discret:LM78LXX
- added C8: 330nF, Capacitors_SMD:C_0805_HandSoldering, B.Cu at (170.2, 104.1)
- added C9: 100nF, Capacitors_SMD:C_0805_HandSoldering, B.Cu at (166.4, 109.2)
- added P10: POWER, Pin_Headers:Pin_Header_Straight_1x02, F.Cu at (163.8, 116.8)
- DS1: footprint Socket_Strips:Socket_Strip_Straight_1x16 -> display-lcd:TUXGR_16X2_R2
- P1: value MA -> MP
- P6: value 5V -> SENSOR; footprint Socket_Strips:Socket_Strip_Straight_1x02 -> Pin_Headers:Pin_Header_Straight_1x09
- P7: value 12V -> 5V
- P8: value SERIAL -> 12V
- P9: value POWER -> SERIAL; footprint Pin_Headers:Pin_Header_Straight_1x02 -> Pin_Headers:Pin_Header_Straight_1x03
- R6: footprint Resistors_SMD:R_0805_HandSoldering -> Resistors_ThroughHole:Resistor_Horizontal_RM15mm; moved to F.Cu
- RV1: footprint Potentiometers:Potentiometer_Trimmer-Suntan-TSR-3386P -> Potentiometers:Potentiometer_Triwood_RM-065
- U1: value TCRT5000 -> LM7805; footprint TCRT5000:TCRT5000 -> Discret:LM78XX-TO92
- U2: value TCRT5000 -> 78L33; footprint TCRT5000:TCRT5000 -> Discret:LM78XX-TO92
- moved U1 141.1 mm to (168.9, 109.2), turned to 225 degrees
- moved U2 137.3 mm to (163.8, 109.2), turned to 45 degrees
- moved P7 110.3 mm to (158.8, 119.4), turned to 270 degrees
- moved C7 102.9 mm to (162.6, 104.1)
- moved P1 97.6 mm to (149.9, 115.6)
- moved P9 85.2 mm to (125.7, 111.8)
- moved C6 57.2 mm to (174.0, 109.2), turned to 90 degrees
- moved P8 43.6 mm to (168.9, 118.1), turned to 270 degrees
- moved RV1 43.5 mm to (178.4, 113.7), turned to 0 degrees
- moved P6 41.9 mm to (100.3, 68.6)
- moved R6 31.8 mm to (157.5, 78.1), turned to 180 degrees
- moved DS1 14.2 mm to (158.8, 83.8)
- moved C4 3.81 mm to (109.2, 97.8)
- turned L1 to 180 degrees
- turned R7 to 90 degrees
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Connections:
- C6 pad 1: /PowerSupply/VCC -> /MotorDriver/+12V
- C7 pad 1: /Debugger/+3.3V -> /Controller/VCC
- P2 pad 1: /Controller/PWM01 -> /Controller/PWM02
- P3 pad 1: /Controller/PWM02 -> /Controller/PWM01
- P6 pad 1: /PowerSupply/VCC -> GND
- P6 pad 2: GND -> /Controller/VCC
- P7 pad 1: /MotorDriver/+12V -> Net-(P7-Pad1)
- P8 pad 1: /Controller/TX -> /MotorDriver/+12V
- P8 pad 2: /Controller/RX -> GND
- P8 pad 3: GND -> Net-(P7-Pad1)
- P9 pad 1: /Debugger/+3.3V -> /Controller/TX
- P9 pad 2: GND -> /Controller/RX
- RV1 pad 1: /Controller/VCC -> GND
- RV1 pad 3: GND -> /Controller/VCC
Routing:
- net GND: track 0.00 -> 295.9 mm
- net /Controller/VCC: track 0.00 -> 230.9 mm, vias 0 -> 5
- net /MotorDriver/+12V: track 0.00 -> 53.9 mm, vias 0 -> 2
- net /Controller/RST: track 0.00 -> 41.6 mm
- net /Controller/MA2: track 0.00 -> 23.2 mm, vias 0 -> 2
- net /Controller/MA1: track 0.00 -> 20.8 mm, vias 0 -> 2
- net /Controller/ADC4: track 0.00 -> 20.3 mm
- net /Controller/ADC3: track 0.00 -> 20.3 mm
- net /Controller/ADC2: track 0.00 -> 20.3 mm
- net /Controller/ADC1: track 0.00 -> 20.3 mm
- net /Controller/ADC0: track 0.00 -> 20.3 mm
- net /Controller/PWM02: track 0.00 -> 15.0 mm
- net /Controller/PWM01: track 0.00 -> 11.4 mm
- net /Controller/MB2: track 0.00 -> 11.4 mm
- net /Controller/MB1: track 0.00 -> 11.4 mm
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Other:
- net class singal added: clearance 0.2, trace_width 0.8, via_dia 0.6, via_drill 0.4
- rule trace_min: 0.2 -> 0.1

Commit message: update
Parts:
- added MountingHole_2-5mm: VAL**, Mounting_Holes:MountingHole_2-5mm, F.Cu at (184.2, 61.6)
- added MountingHole_2-5mm: VAL**, Mounting_Holes:MountingHole_2-5mm, F.Cu at (184.2, 120.0)
- added MountingHole_2-5mm: VAL**, Mounting_Holes:MountingHole_2-5mm, F.Cu at (78.7, 61.6)
- added MountingHole_2-5mm: VAL**, Mounting_Holes:MountingHole_2-5mm, F.Cu at (78.7, 120.0)
- moved P10 6.48 mm to (157.5, 115.6)
- moved C6 6.48 mm to (167.6, 108.0)
- moved P1 6.48 mm to (143.5, 114.3)
- moved U2 6.48 mm to (157.5, 108.0)
- moved P5 6.48 mm to (105.4, 110.5)
- moved P9 6.48 mm to (119.4, 110.5)
- moved C2 6.48 mm to (119.4, 94.0)
- moved D3 6.48 mm to (91.4, 111.8)
- moved IC1 6.48 mm to (110.5, 95.2)
- moved R3 6.48 mm to (101.6, 82.5)
- moved R9 6.48 mm to (91.4, 106.7)
- moved SW1 6.48 mm to (82.5, 106.7)
- moved SW2 6.48 mm to (101.6, 76.2)
- moved X1 6.48 mm to (115.6, 97.8)
- moved C4 6.48 mm to (102.9, 96.5)
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Routing:
- net GND: track 295.9 -> 9.71 mm
- net /Controller/VCC: track 230.9 -> 234.4 mm
- net /Controller/CONTRAS: track 5.08 -> 7.62 mm
- net /MotorDriver/+12V: track 53.9 -> 55.8 mm
- net (no net): track 1.80 -> 0.00 mm
- net /Controller/LCD_E: track 2.54 -> 3.81 mm
- net /Controller/LCD_RS: track 5.44 -> 6.71 mm
- net /Controller/LCD_D7: track 5.44 -> 6.71 mm
- net /Controller/LCD_D6: track 5.44 -> 6.71 mm
- net /Controller/LCD_D5: track 5.44 -> 6.71 mm
- net /Controller/LCD_D4: track 5.44 -> 6.71 mm
- added copper zone on B.Cu, net GND
